File: Liam-Sandra-Peregrine-Tim/foe-scale.brd (EAGLE design)
At the start: 96.2 x 67.3 mm, 49 parts, among them U1 LM311, U2 SAMD21E

Commit message: eagle why you gotta be that way?
Parts:
- moved U$8 2.54 mm to (67.3, 17.8)
Routing:
- net CS-PA19: track 21.8 -> 44.3 mm
- net DI-PA18: track 21.7 -> 42.2 mm
- net DO-PA16: track 20.5 -> 39.4 mm, vias 0 -> 2
- net RST: track 43.2 -> 46.1 mm
- net DGND: track 70.8 -> 72.2 mm
- net CLK-PA17: track 21.1 -> 22.0 mm, vias 0 -> 2
- net +3V3: track 172.2 -> 172.9 mm
Other:
- board text added: "Level Shifter"
- board text added: "MicroSD"
- board text added: "MicroUSB"
