File: Liam-Sandra-Peregrine-Tim/foe-scale.sch (EAGLE design)
At the start: 24 parts, among them U1 LM311

Commit message: got most of the parts for the schematic in
Parts:
- added C6, C7: 100nF, rcl:C-EUC0805K
- added C8: .1uF, rcl:C-EUC0805K
- added C9: 10nF, rcl:C-EUC0805K
- added D1: (no value), foe-scale:D1213A-DIODE-ARRAY
- added DBG1: DEBUGHEAD, foe-scale:DEBUGHEAD
- added R10, R11: 10k, resistor:R-US_R0805
- added R12: 100k, resistor:R-US_R0805
- added R13: 0, resistor:R-US_R0805
- added U$10: RGBLED, foe-scale:RGBLED
- added U$11, U$12: PUSHBTN, foe-scale:PUSHBTN
- added U$13: MICRO-USB-CONNECTOR, foe-scale:MICRO-USB-CONNECTOR
- added U2: SAMD21E, foe-scale:SAMD21E
- added U3: 3.3V_AS1363, foe-scale:3.3V_AS1363
Connections:
- net N$2 renamed V+
- net N$3 renamed V-
- net N$31 renamed /SAMPLE-PA01
- net N$32 renamed HYS-PA02
- net N$41 renamed SDO-PA09
- net N$42 renamed CONV-PA10
- net N$43 renamed SCK-PA08
- new net N$2: U$12.2, U2.PA28
- new net N$3: U$11.2, U2.PA27
- new net N$31: U2.RESETN
- new net N$32: C6.2
- new net N$41: U$13.GND
- new net N$42: D1.CH2, U$13.D-
- new net N$43: D1.CH1, U$13.D+
- new net N$44: U2.GND2
- new net N$45: C7.2, U2.VDDCORE
- new net N$46: C7.1
- new net N$47: U$10.A
- new net N$48: U$10.4-GREEN, U2.PA03
- new net N$49: U$10.3-BLUE, U2.PA04
- new net N$50: U$10.1-RED, U2.PA05
- new net N$51: U2.PA16
- new net N$52: U2.PA17
- new net N$53: U2.PA18
- new net N$54: U2.PA19
- new net N$55: U2.PA08
- new net N$56: U2.PA09
- new net N$57: U2.PA10
- new net N$58: U2.PA11
- new net N$59: U2.VDDIN
- new net N$60: U2.GND
- new net N$61: U2.PA02
- new net N$62: U2.VDDANA
- new net N$63: C8.1, R11.1, U3.IN
- new net N$64: R11.2, U3.EN
- new net N$65: R12.1
- new net N$66: C8.2
- new net N$67: C9.1, U3.SET
- new net N$68: C9.2, U3.OUT
- new net N$69: DBG1.VTREF
- new net N$70: R12.2, U3.POK
- new net N$71: U3.GND
- new net N$72: R13.2
- new net N$73: R13.1
- new net N$74: DBG1.GND1, DBG1.GND2
- new net N$75: DBG1.SWDIO
- new net N$76: DBG1.SWDCLK
- new net N$77: D1.V_N
- new net N$78: D1.V_P
- new net N$79: DBG1.RSTB
- new net RST: C6.1, R10.1
- new net SWDCLK: U2.PA30
- new net SWDIO: U2.PA31
- new net USB_D+_PA25: U2.PA25
- new net USB_D-_PA24: U2.PA24
- net DGND: now also U$11.1, U$12.1
- net N$10: no longer U$3G$2.AIN+
- net N$16: now also U$2.REF, U$3G$1.AIN-, U$3G$1.OUT; no longer U$3G$2.AIN-, U$3G$2.OUT
- net N$9: now also R10.2; no longer U$2.REF, U$3G$1.AIN-, U$3G$1.OUT
Other:
- note added: "Reset Circuitry"
- note added: "ferrite bead"
- note removed: "+5v"
- note removed: "/SAMPLE-PA11"
- note removed: "3.3V"
- note removed: "CONV-PA10"
- note removed: "HYS-PA02"
- note removed: "SCK-PA08"
- note removed: "SDO-PA09"
- note removed: "V+"
- note removed: "V-"

Commit message: finished up schematic
Parts:
- U$8: value SDCARD_JACK -> (none); device test:SDCARD_JACK -> foe-scale:SDCARD_JACK
- U$9: device test:RED_LED -> foe-scale:RED_LED
Connections:
- net N$40 renamed +3.3V
- removed net /SAMPLE-PA01: U1.COUT
- removed net N$1: U$1.1
- removed net N$11: R3.1
- removed net N$12: R2.2
- removed net N$13: U$3G$3.V+
- removed net N$14: U$3G$3.V-
- removed net N$15: U$2.+VS
- removed net N$17: C2.2
- removed net N$21: C1.2
- removed net N$22: R7.1
- removed net N$24: R8.2
- removed net N$25: C4.2
- removed net N$26: U1.EOUT
- removed net N$28: C5.2
- removed net N$29: U1.VCC
- removed net N$30: U1.VDD
- removed net N$31: U2.RESETN
- removed net N$32: C6.2
- removed net N$33: U$6.GND, U$6.IN-
- removed net N$37: U$6.VCC
- removed net N$38: U$7.V_L
- removed net N$39: U$7.GND, U$7.IV_L4
- removed net N$4: U$1.4
- removed net N$41: U$13.GND
- removed net N$42: D1.CH2, U$13.D-
- removed net N$43: D1.CH1, U$13.D+
- removed net N$44: U2.GND2
- removed net N$47: U$10.A
- removed net N$51: U2.PA16
- removed net N$52: U2.PA17
- removed net N$53: U2.PA18
- removed net N$54: U2.PA19
- removed net N$55: U2.PA08
- removed net N$56: U2.PA09
- removed net N$57: U2.PA10
- removed net N$58: U2.PA11
- removed net N$59: U2.VDDIN
- removed net N$60: U2.GND
- removed net N$61: U2.PA02
- removed net N$62: U2.VDDANA
- removed net N$63: C8.1, R11.1, U3.IN
- removed net N$66: C8.2
- removed net N$68: C9.2, U3.OUT
- removed net N$69: DBG1.VTREF
- removed net N$71: U3.GND
- removed net N$72: R13.2
- removed net N$73: R13.1
- removed net N$74: DBG1.GND1, DBG1.GND2
- removed net N$75: DBG1.SWDIO
- removed net N$76: DBG1.SWDCLK
- removed net N$77: D1.V_N
- removed net N$78: D1.V_P
- removed net N$79: DBG1.RSTB
- removed net N$8: U$2.–VS
- new net /SAMPLE-PA11: U1.COUT, U2.PA11
- net +5V: now also C8.1, D1.V_P, R11.1, R2.2, R7.1, U$1.1, U$2.+VS, U$3G$3.V+, U$6.VCC, U$7.V_L, U1.VDD, U3.IN; no longer U$9.P+
- net 3.3V: now also C9.2, DBG1.VTREF, U$10.A, U$8.VDD, U2.VDDANA, U2.VDDIN, U3.OUT; no longer U$8.P4/VDD
- net AGND: now also C1.2, C2.2, C4.2, C5.2, R13.2, R3.1, R8.2, U$1.4, U$2.–VS, U$3G$3.V-, U$6.GND, U$6.IN-, U$7.GND, U$7.IV_L4, U1.EOUT, U1.VCC; no longer U$9.P-
- net CLK-PA17: now also U$8.CLK, U2.PA17; no longer U$8.P5/SCLK
- net CONV-PA10: now also U2.PA10
- net CS-PA19: now also U$8.CD, U2.PA19; no longer U$8.P2/CS
- net DGND: now also C6.2, C8.2, D1.V_N, DBG1.GND1, DBG1.GND2, R13.1, U$13.GND, U$8.VSS, U2.GND, U2.GND2, U3.GND; no longer U$8.P6/VSS
- net DI-PA18: now also U$8.CMD, U2.PA18; no longer U$8.P3/DI
- net DO-PA16: now also U$8.DAT0, U2.PA16; no longer U$8.P7/DO
- net HYS-PA02: now also U2.PA02
- net RST: now also DBG1.RSTB, U2.RESETN
- net SCK-PA08: now also U2.PA08
- net SDO-PA09: now also U2.PA09
- net SWDCLK: now also DBG1.SWDCLK
- net SWDIO: now also DBG1.SWDIO
- net USB_D+_PA25: now also D1.CH1, U$13.D+
- net USB_D-_PA24: now also D1.CH2, U$13.D-
Other:
- note removed: "AGND"

Commit message: added some labels, consolidated space, moved some parts around to generate dividing plane
Parts:
- removed U3: 3.3V_AS1363, foe-scale:3.3V_AS1363
- added AS1363: (no value), foe-scale:3.3V_AS1363
Connections:
- net +5V: now also AS1363.IN; no longer U3.IN
- net 3.3V: now also AS1363.OUT; no longer U3.OUT
- net DGND: now also AS1363.GND; no longer U3.GND
- net N$64: now also AS1363.EN; no longer U3.EN
- net N$67: now also AS1363.SET; no longer U3.SET
- net N$70: now also AS1363.POK; no longer U3.POK
Changed lines of the file:
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@@
 <?xml version="1.0" encoding="utf-8"?>
 <!DOCTYPE eagle SYSTEM "eagle.dtd">
-<eagle version="7.4.0">
+<eagle version="7.5.0">
 <drawing>
 <settings>
@@
 <grid distance="0.1" unitdist="inch" unit="inch" style="lines" multiple="1" display="no" altdistance="0.01" altunitdist="inch" altunit="inch"/>
 <layers>
-<layer number="1" name="Top" color="4" fill="1" visible="no" active="no"/>
-<layer number="16" name="Bottom" color="1" fill="1" visible="no" active="no"/>
-<layer number="17" name="Pads" color="2" fill="1" visible="no" active="no"/>
-<layer number="18" name="Vias" color="2" fill="1" visible="no" active="no"/>
-<layer number="19" name="Unrouted" color="6" fill="1" visible="no" active="no"/>
-<layer number="20" name="Dimension" color="15" fill="1" visible="no" active="no"/>
-<layer number="21" name="tPlace" color="7" fill="1" visible="no" active="no"/>
-<layer number="22" name="bPlace" color="7" fill="1" visible="no" active="no"/>
-<layer number="23" name="tOrigins" color="15" fill="1" visible="no" active="no"/>
-<layer number="24" name="bOrigins" color="15" fill="1" visible="no" active="no"/>
-<layer number="25" name="tNames" color="7" fill="1" visible="no" active="no"/>
-<layer number="26" name="bNames" color="7" fill="1" visible="no" active="no"/>
-<layer number="27" name="tValues" color="7" fill="1" visible="no" active="no"/>
-<layer number="28" name="bValues" color="7" fill="1" visible="no" active="no"/>
+<layer number="1" name="Top" color="4" fill="1" visible="yes" active="no"/>
+<layer number="16" name="Bottom" color="1" fill="1" visible="yes" active="no"/>
+<layer number="17" name="Pads" color="2" fill="1" visible="yes" active="no"/>
+<layer number="18" name="Vias" color="2" fill="1" visible="yes" active="no"/>
+<layer number="19" name="Unrouted" color="6" fill="1" visible="yes" active="no"/>
+<layer number="20" name="Dimension" color="15" fill="1" visible="yes" active="no"/>
+<layer number="21" name="tPlace" color="7" fill="1" visible="yes" active="no"/>
+<layer number="22" name="bPlace" color="7" fill="1" visible="yes" active="no"/>
+<layer number="23" name="tOrigins" color="15" fill="1" visible="yes" active="no"/>
+<layer number="24" name="bOrigins" color="15" fill="1" visible="yes" active="no"/>
+<layer number="25" name="tNames" color="7" fill="1" visible="yes" active="no"/>
+<layer number="26" name="bNames" color="7" fill="1" visible="yes" active="no"/>
+<layer number="27" name="tValues" color="7" fill="1" visible="yes" active="no"/>
+<layer number="28" name="bValues" color="7" fill="1" visible="yes" active="no"/>
 <layer number="29" name="tStop" color="7" fill="3" visible="no" active="no"/>
 <layer number="30" name="bStop" color="7" fill="6" visible="no" active="no"/>
@@
 <layer number="35" name="tGlue" color="7" fill="4" visible="no" active="no"/>
 <layer number="36" name="bGlue" color="7" fill="5" visible="no" active="no"/>
-<layer number="37" name="tTest" color="7" fill="1" visible="no" active="no"/>
-<layer number="38" name="bTest" color="7" fill="1" visible="no" active="no"/>
+<layer number="37" name="tTest" color="7" fill="1" visible="yes" active="no"/>
+<layer number="38" name="bTest" color="7" fill="1" visible="yes" active="no"/>
 <layer number="39" name="tKeepout" color="4" fill="11" visible="no" active="no"/>
 <layer number="40" name="bKeepout" color="1" fill="11" visible="no" active="no"/>
@@
 <layer number="44" name="Drills" color="7" fill="1" visible="no" active="no"/>
 <layer number="45" name="Holes" color="7" fill="1" visible="no" active="no"/>
-<layer number="46" name="Milling" color="3" fill="1" visible="no" active="no"/>
-<layer number="47" name="Measures" color="7" fill="1" visible="no" active="no"/>
-<layer number="48" name="Document" color="7" fill="1" visible="no" active="no"/>
-<layer number="49" name="Reference" color="7" fill="1" visible="no" active="no"/>
-<layer number="51" name="tDocu" color="7" fill="1" visible="no" active="no"/>
-<layer number="52" name="bDocu" color="7" fill="1" visible="no" active="no"/>
+<layer number="46" name="Milling" color="3" fill="1" visible="yes" active="no"/>
+<layer number="47" name="Measures" color="7" fill="1" visible="yes" active="no"/>
+<layer number="48" name="Document" color="7" fill="1" visible="yes" active="no"/>
+<layer number="49" name="Reference" color="7" fill="1" visible="yes" active="no"/>
+<layer number="51" name="tDocu" color="7" fill="1" visible="yes" active="no"/>
+<layer number="52" name="bDocu" color="7" fill="1" visible="yes" active="no"/>
 <layer number="90" name="Modules" color="5" fill="1" visible="yes" active="yes"/>
 <layer number="91" name="Nets" color="2" fill="1" visible="yes" active="yes"/>
@@
 <part name="U$10" library="foe-scale" deviceset="RGBLED" device=""/>
 <part name="U$13" library="foe-scale" deviceset="MICRO-USB-CONNECTOR" device=""/>
-<part name="U3" library="foe-scale" deviceset="3.3V_AS1363" device=""/>
+<part name="AS1363" library="foe-scale" deviceset="3.3V_AS1363" device=""/>
 <part name="R11" library="resistor" deviceset="R-US_" device="R0805" value="10k"/>
 <part name="C8" library="rcl" deviceset="C-EU" device="C0805K" value=".1uF"/>
@@
 <instance part="C7" gate="G$1" x="43.18" y="-38.1"/>
 <instance part="U$10" gate="G$1" x="-7.62" y="-111.76"/>
-<instance part="U$13" gate="G$1" x="210.82" y="-25.4"/>
-<instance part="U3" gate="G$1" x="160.02" y="5.08"/>
+<instance part="U$13" gate="G$1" x="215.9" y="-25.4"/>
+<instance part="AS1363" gate="AS1363" x="160.02" y="5.08"/>
 <instance part="R11" gate="G$1" x="134.62" y="10.16" rot="R270"/>
 <instance part="C8" gate="G$1" x="127" y="15.24"/>
@@
 </segment>
 <segment>
-<pinref part="U3" gate="G$1" pin="GND"/>
+<pinref part="AS1363" gate="AS1363" pin="GND"/>
 <wire x1="172.72" y1="-2.54" x2="182.88" y2="-2.54" width="0.1524" layer="91"/>
 <wire x1="182.88" y1="-2.54" x2="182.88" y2="-12.7" width="0.1524" layer="91"/>
@@
 <segment>
 <pinref part="U$13" gate="G$1" pin="GND"/>
-<wire x1="210.82" y1="-7.62" x2="241.3" y2="-7.62" width="0.1524" layer="91"/>
+<wire x1="215.9" y1="-7.62" x2="241.3" y2="-7.62" width="0.1524" layer="91"/>
 <wire x1="241.3" y1="-7.62" x2="241.3" y2="-15.24" width="0.1524" layer="91"/>
 <label x="241.3" y="-10.16" size="1.778" layer="95" rot="R180"/>
@@
 <pinref part="C9" gate="G$1" pin="2"/>
 <wire x1="190.5" y1="5.08" x2="198.12" y2="5.08" width="0.1524" layer="91"/>
-<pinref part="U3" gate="G$1" pin="OUT"/>
+<pinref part="AS1363" gate="AS1363" pin="OUT"/>
 <wire x1="172.72" y1="12.7" x2="198.12" y2="12.7" width="0.1524" layer="91"/>
 <wire x1="198.12" y1="12.7" x2="198.12" y2="5.08" width="0.1524" layer="91"/>
@@
 <segment>
 <pinref part="R11" gate="G$1" pin="1"/>
-<pinref part="U3" gate="G$1" pin="IN"/>
+<pinref part="AS1363" gate="AS1363" pin="IN"/>
 <wire x1="134.62" y1="15.24" x2="147.32" y2="15.24" width="0.1524" layer="91"/>
 <wire x1="147.32" y1="15.24" x2="147.32" y2="12.7" width="0.1524" layer="91"/>
@@
 <segment>
 <pinref part="U$13" gate="G$1" pin="D-"/>
-<wire x1="210.82" y1="-22.86" x2="231.14" y2="-22.86" width="0.1524" layer="91"/>
+<wire x1="215.9" y1="-22.86" x2="231.14" y2="-22.86" width="0.1524" layer="91"/>
 <wire x1="231.14" y1="-22.86" x2="231.14" y2="-30.48" width="0.1524" layer="91"/>
 <wire x1="231.14" y1="-30.48" x2="289.56" y2="-30.48" width="0.1524" layer="91"/>
@@
 <segment>
 <pinref part="U$13" gate="G$1" pin="D+"/>
-<wire x1="210.82" y1="-17.78" x2="246.38" y2="-17.78" width="0.1524" layer="91"/>
+<wire x1="215.9" y1="-17.78" x2="246.38" y2="-17.78" width="0.1524" layer="91"/>
 <wire x1="246.38" y1="-17.78" x2="246.38" y2="-22.86" width="0.1524" layer="91"/>
 <pinref part="D1" gate="G$1" pin="CH1"/>
@@
 <pinref part="R11" gate="G$1" pin="2"/>
 <wire x1="134.62" y1="5.08" x2="147.32" y2="5.08" width="0.1524" layer="91"/>
-<pinref part="U3" gate="G$1" pin="EN"/>
+<pinref part="AS1363" gate="AS1363" pin="EN"/>
 </segment>
 </net>
@@
 <segment>
 <pinref part="C9" gate="G$1" pin="1"/>
-<pinref part="U3" gate="G$1" pin="SET"/>
+<pinref part="AS1363" gate="AS1363" pin="SET"/>
 <wire x1="182.88" y1="5.08" x2="172.72" y2="5.08" width="0.1524" layer="91"/>
 </segment>
@@
 <segment>
 <pinref part="R12" gate="G$1" pin="2"/>
-<pinref part="U3" gate="G$1" pin="POK"/>
+<pinref part="AS1363" gate="AS1363" pin="POK"/>
 <wire x1="142.24" y1="-2.54" x2="147.32" y2="-2.54" width="0.1524" layer="91"/>
 </segment>

Commit message: minor changes
Connections:
- removed net +3.3V: U$7.V_CC
- removed net N$9: R10.2
- net 3.3V: now also R10.2, U$7.V_CC
- net SCK-PA08: no longer U$7.IV_CC1
Changed lines of the file:
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@@
 <?xml version="1.0" encoding="utf-8"?>
 <!DOCTYPE eagle SYSTEM "eagle.dtd">
-<eagle version="7.5.0">
+<eagle version="7.4.0">
 <drawing>
 <settings>
@@
 <grid distance="0.1" unitdist="inch" unit="inch" style="lines" multiple="1" display="no" altdistance="0.01" altunitdist="inch" altunit="inch"/>
 <layers>
-<layer number="1" name="Top" color="4" fill="1" visible="yes" active="no"/>
-<layer number="16" name="Bottom" color="1" fill="1" visible="yes" active="no"/>
-<layer number="17" name="Pads" color="2" fill="1" visible="yes" active="no"/>
-<layer number="18" name="Vias" color="2" fill="1" visible="yes" active="no"/>
-<layer number="19" name="Unrouted" color="6" fill="1" visible="yes" active="no"/>
-<layer number="20" name="Dimension" color="15" fill="1" visible="yes" active="no"/>
-<layer number="21" name="tPlace" color="7" fill="1" visible="yes" active="no"/>
-<layer number="22" name="bPlace" color="7" fill="1" visible="yes" active="no"/>
-<layer number="23" name="tOrigins" color="15" fill="1" visible="yes" active="no"/>
-<layer number="24" name="bOrigins" color="15" fill="1" visible="yes" active="no"/>
-<layer number="25" name="tNames" color="7" fill="1" visible="yes" active="no"/>
-<layer number="26" name="bNames" color="7" fill="1" visible="yes" active="no"/>
-<layer number="27" name="tValues" color="7" fill="1" visible="yes" active="no"/>
-<layer number="28" name="bValues" color="7" fill="1" visible="yes" active="no"/>
+<layer number="1" name="Top" color="4" fill="1" visible="no" active="no"/>
+<layer number="16" name="Bottom" color="1" fill="1" visible="no" active="no"/>
+<layer number="17" name="Pads" color="2" fill="1" visible="no" active="no"/>
+<layer number="18" name="Vias" color="2" fill="1" visible="no" active="no"/>
+<layer number="19" name="Unrouted" color="6" fill="1" visible="no" active="no"/>
+<layer number="20" name="Dimension" color="15" fill="1" visible="no" active="no"/>
+<layer number="21" name="tPlace" color="7" fill="1" visible="no" active="no"/>
+<layer number="22" name="bPlace" color="7" fill="1" visible="no" active="no"/>
+<layer number="23" name="tOrigins" color="15" fill="1" visible="no" active="no"/>
+<layer number="24" name="bOrigins" color="15" fill="1" visible="no" active="no"/>
+<layer number="25" name="tNames" color="7" fill="1" visible="no" active="no"/>
+<layer number="26" name="bNames" color="7" fill="1" visible="no" active="no"/>
+<layer number="27" name="tValues" color="7" fill="1" visible="no" active="no"/>
+<layer number="28" name="bValues" color="7" fill="1" visible="no" active="no"/>
 <layer number="29" name="tStop" color="7" fill="3" visible="no" active="no"/>
 <layer number="30" name="bStop" color="7" fill="6" visible="no" active="no"/>
@@
 <layer number="35" name="tGlue" color="7" fill="4" visible="no" active="no"/>
 <layer number="36" name="bGlue" color="7" fill="5" visible="no" active="no"/>
-<layer number="37" name="tTest" color="7" fill="1" visible="yes" active="no"/>
-<layer number="38" name="bTest" color="7" fill="1" visible="yes" active="no"/>
+<layer number="37" name="tTest" color="7" fill="1" visible="no" active="no"/>
+<layer number="38" name="bTest" color="7" fill="1" visible="no" active="no"/>
 <layer number="39" name="tKeepout" color="4" fill="11" visible="no" active="no"/>
 <layer number="40" name="bKeepout" color="1" fill="11" visible="no" active="no"/>
@@
 <layer number="44" name="Drills" color="7" fill="1" visible="no" active="no"/>
 <layer number="45" name="Holes" color="7" fill="1" visible="no" active="no"/>
-<layer number="46" name="Milling" color="3" fill="1" visible="yes" active="no"/>
-<layer number="47" name="Measures" color="7" fill="1" visible="yes" active="no"/>
-<layer number="48" name="Document" color="7" fill="1" visible="yes" active="no"/>
-<layer number="49" name="Reference" color="7" fill="1" visible="yes" active="no"/>
-<layer number="51" name="tDocu" color="7" fill="1" visible="yes" active="no"/>
-<layer number="52" name="bDocu" color="7" fill="1" visible="yes" active="no"/>
+<layer number="46" name="Milling" color="3" fill="1" visible="no" active="no"/>
+<layer number="47" name="Measures" color="7" fill="1" visible="no" active="no"/>
+<layer number="48" name="Document" color="7" fill="1" visible="no" active="no"/>
+<layer number="49" name="Reference" color="7" fill="1" visible="no" active="no"/>
+<layer number="51" name="tDocu" color="7" fill="1" visible="no" active="no"/>
+<layer number="52" name="bDocu" color="7" fill="1" visible="no" active="no"/>
 <layer number="90" name="Modules" color="5" fill="1" visible="yes" active="yes"/>
 <layer number="91" name="Nets" color="2" fill="1" visible="yes" active="yes"/>
@@
 </segment>
 </net>
-<net name="+3.3V" class="0">
-<segment>
-<pinref part="U$7" gate="G$1" pin="V_CC"/>
-<wire x1="434.34" y1="114.3" x2="441.96" y2="114.3" width="0.1524" layer="91"/>
-<wire x1="441.96" y1="114.3" x2="441.96" y2="132.08" width="0.1524" layer="91"/>
-<label x="441.96" y="127" size="1.778" layer="95"/>
-</segment>
-</net>
 <net name="N$34" class="0">
 <segment>
@@
 </net>
 <net name="SCK-PA08" class="0">
-<segment>
-<pinref part="U$7" gate="G$1" pin="IV_CC1"/>
-<wire x1="434.34" y1="109.22" x2="454.66" y2="109.22" width="0.1524" layer="91"/>
-<label x="447.04" y="109.22" size="1.778" layer="95"/>
-</segment>
 <segment>
 <pinref part="U2" gate="G$1" pin="PA08"/>
@@
 <label x="101.6" y="5.08" size="1.778" layer="95"/>
 <wire x1="83.82" y1="5.08" x2="109.22" y2="5.08" width="0.1524" layer="91"/>
-<label x="-27.94" y="27.94" size="1.778" layer="95"/>
 <label x="127" y="0" size="1.778" layer="95"/>
 </segment>
@@
 <wire x1="-12.7" y1="-121.92" x2="-12.7" y2="-132.08" width="0.1524" layer="91"/>
 <label x="-12.7" y="-129.54" size="1.778" layer="95" rot="R90"/>
+</segment>
+<segment>
+<pinref part="U$7" gate="G$1" pin="V_CC"/>
+<wire x1="434.34" y1="114.3" x2="439.42" y2="114.3" width="0.1524" layer="91" style="dashdot"/>
+<wire x1="439.42" y1="114.3" x2="439.42" y2="127" width="0.1524" layer="91" style="dashdot"/>
+<label x="439.42" y="124.46" size="1.778" layer="95"/>
+</segment>
+<segment>
+<pinref part="R10" gate="G$1" pin="2"/>
+<wire x1="-27.94" y1="22.86" x2="-27.94" y2="33.02" width="0.1524" layer="91" style="dashdot"/>
+<label x="-27.94" y="30.48" size="1.778" layer="95"/>
 </segment>
 </net>
@@
 </segment>
 </net>
-<net name="N$9" class="0">
-<segment>
-<pinref part="R10" gate="G$1" pin="2"/>
-<wire x1="-27.94" y1="22.86" x2="-27.94" y2="30.48" width="0.1524" layer="91"/>
-</segment>
-</net>

Commit message: added power and gnd connections
Connections:
- removed net 3.3V: AS1363.OUT, C9.2, DBG1.VTREF, R10.2, U$10.A, U$7.V_CC, U$8.VDD, U2.VDDANA, U2.VDDIN
- removed net N$46: C7.1
- removed net N$65: R12.1
- new net +3V3: AS1363.OUT, C9.2, DBG1.VTREF, R10.2, R12.1, U$10.A, U$7.V_CC, U$8.VDD, U2.VDDANA, U2.VDDIN
- new net TESTTESTTEST: C4.2
- net AGND: no longer C4.2
- net DGND: now also C7.1
- net SCK-PA08: now also U$7.IV_CC1

Commit message: made a few changes to layout
Parts:
- added R14, R15: 15, resistor:R-US_R0805
- added R16: 70, resistor:R-US_R0805
- U$11, U$12: value PUSHBTN -> BUTTON_THRU; device foe-scale:PUSHBTN -> foe-scale:BUTTON_THRU
Connections:
- new net N$1: R14.1, U2.PA03
- new net N$4: R15.1, U2.PA04
- new net N$8: R16.1, U2.PA05
- net AGND: no longer U$7.GND, U$7.IV_L4
- net DGND: now also U$7.GND, U$7.IV_L4
- net N$48: now also R14.2; no longer U2.PA03
- net N$49: now also R15.2; no longer U2.PA04
- net N$50: now also R16.2; no longer U2.PA05
