File: final_project_scott_liam_tim_peregrine/syma-wireless-charger.sch (EAGLE design)
At the start: 3 parts, among them U1 SAMD21E

Commit message: worked on the schematic a bit
Parts:
- removed U$2: LTC4120-4.2V, foe-scale:LTC4120-4.2V
- added C1, C3: (no value), resistor:C-EUC0805K
- added C2, C5: 100nF, resistor:C-EUC0805K
- added C4: 10nF, resistor:C-EUC0805K
- added DBG1: DEBUGHEAD, foe-scale:DEBUGHEAD
- added R1, R4: (no value), resistor:R-US_R0805
- added R2, R3: 10k, resistor:R-US_R0805
- added U$3: 1X02, foe-scale:1X02
- added U2: (no value), foe-scale:3.3V_AS1363
Connections:
- new net +5V: C3.1, R2.2, U$3.P$1
- new net GND: C2.1, C3.2, C5.2, DBG1.GND1, DBG1.GND2, U$3.P$2, U1.GND, U1.GND2, U2.GND
- new net N$1: C2.2, U1.VDDCORE
- new net N$2: R3.2, U2.POK
- new net N$3: R2.1, U2.EN
- new net N$5: C4.1, U2.SET
- new net RST: C5.1, DBG1.RSTB, R4.1, U1.RESETN
- new net SWDCLK-PA30: DBG1.SWDCLK, U1.PA30
- new net SWDIO-PA31: DBG1.SWDIO, U1.PA31
- new net VDD: C4.2, DBG1.VTREF, R3.1, R4.2, U1.VDDANA, U1.VDDIN, U2.OUT

Commit message: started tranmitter circuit
Parts:
- added C6, C7: 100n, rcl:C-EUC0805
- added R10: 7.87k, rcl:R-US_R0805
- added R11, R14, R15, R5: (no value), rcl:R-US_R0805
- added R12: 5.23k, rcl:R-US_R0805
- added R13, R7, R9: 100k, rcl:R-US_R0805
- added R6: 348k, rcl:R-US_R0805
- added R8: 59k, rcl:R-US_R0805
- added U$2: BAS521, foe-scale:BAS521
- C1: value (none) -> 10n; device resistor:C-EUC0805K -> rcl:C-EUC0805
Connections:
- new net N$10: C7.1, R13.2, U$2.CATHODE
- new net N$11: C7.2, R12.1
- new net N$12: U$1.SW2
- new net N$4: R10.2, R9.1, U$1.DTH
- new net N$6: R7.1, R8.2, U$1.FTH
- new net N$7: U$1.IN1, U$1.IN2
- new net N$8: C1.2, R6.1, U$1.IMON
- new net N$9: C6.2, R12.2, R13.1, U$1.FB
- net GND: now also C1.1, R10.1, R6.2, R8.1, U$1.GND
Other:
- moved on the sheet: C1

Commit message: finished uC
Parts:
- added R16, R18: 15, resistor:R-US_R0805
- added R17: 70, resistor:R-US_R0805
- added U$4: RGBLED, foe-scale:RGBLED
- added U$5: BUZZER, foe-scale:BUZZER
Connections:
- new net ALIGNED: U1.PA03
- new net CARSENSE: U1.PA05
- new net ENVSENSE: U1.PA06
- new net IMON: U1.PA04
- new net N$13: R17.2, U1.PA22
- new net N$14: R18.2, U1.PA19
- new net N$15: R16.2, U1.PA18
- new net N$16: R16.1, U$4.4-GREEN
- new net N$17: R18.1, U$4.3-BLUE
- new net N$18: R17.1, U$4.1-RED
- new net N$19: U$5.+, U1.PA23
- net GND: now also U$5.-
- net VDD: now also U$4.A
Changed lines of the file:
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@@
 <grid distance="0.1" unitdist="inch" unit="inch" style="lines" multiple="1" display="no" altdistance="0.01" altunitdist="inch" altunit="inch"/>
 <layers>
-<layer number="1" name="Top" color="4" fill="1" visible="yes" active="no"/>
-<layer number="16" name="Bottom" color="1" fill="1" visible="yes" active="no"/>
-<layer number="17" name="Pads" color="2" fill="1" visible="yes" active="no"/>
-<layer number="18" name="Vias" color="2" fill="1" visible="yes" active="no"/>
-<layer number="19" name="Unrouted" color="6" fill="1" visible="yes" active="no"/>
-<layer number="20" name="Dimension" color="15" fill="1" visible="yes" active="no"/>
-<layer number="21" name="tPlace" color="7" fill="1" visible="yes" active="no"/>
-<layer number="22" name="bPlace" color="7" fill="1" visible="yes" active="no"/>
-<layer number="23" name="tOrigins" color="15" fill="1" visible="yes" active="no"/>
-<layer number="24" name="bOrigins" color="15" fill="1" visible="yes" active="no"/>
-<layer number="25" name="tNames" color="7" fill="1" visible="yes" active="no"/>
-<layer number="26" name="bNames" color="7" fill="1" visible="yes" active="no"/>
-<layer number="27" name="tValues" color="7" fill="1" visible="yes" active="no"/>
-<layer number="28" name="bValues" color="7" fill="1" visible="yes" active="no"/>
+<layer number="1" name="Top" color="4" fill="1" visible="no" active="no"/>
+<layer number="16" name="Bottom" color="1" fill="1" visible="no" active="no"/>
+<layer number="17" name="Pads" color="2" fill="1" visible="no" active="no"/>
+<layer number="18" name="Vias" color="2" fill="1" visible="no" active="no"/>
+<layer number="19" name="Unrouted" color="6" fill="1" visible="no" active="no"/>
+<layer number="20" name="Dimension" color="15" fill="1" visible="no" active="no"/>
+<layer number="21" name="tPlace" color="7" fill="1" visible="no" active="no"/>
+<layer number="22" name="bPlace" color="7" fill="1" visible="no" active="no"/>
+<layer number="23" name="tOrigins" color="15" fill="1" visible="no" active="no"/>
+<layer number="24" name="bOrigins" color="15" fill="1" visible="no" active="no"/>
+<layer number="25" name="tNames" color="7" fill="1" visible="no" active="no"/>
+<layer number="26" name="bNames" color="7" fill="1" visible="no" active="no"/>
+<layer number="27" name="tValues" color="7" fill="1" visible="no" active="no"/>
+<layer number="28" name="bValues" color="7" fill="1" visible="no" active="no"/>
 <layer number="29" name="tStop" color="7" fill="3" visible="no" active="no"/>
 <layer number="30" name="bStop" color="7" fill="6" visible="no" active="no"/>
@@
 <layer number="35" name="tGlue" color="7" fill="4" visible="no" active="no"/>
 <layer number="36" name="bGlue" color="7" fill="5" visible="no" active="no"/>
-<layer number="37" name="tTest" color="7" fill="1" visible="yes" active="no"/>
-<layer number="38" name="bTest" color="7" fill="1" visible="yes" active="no"/>
+<layer number="37" name="tTest" color="7" fill="1" visible="no" active="no"/>
+<layer number="38" name="bTest" color="7" fill="1" visible="no" active="no"/>
 <layer number="39" name="tKeepout" color="4" fill="11" visible="no" active="no"/>
 <layer number="40" name="bKeepout" color="1" fill="11" visible="no" active="no"/>
@@
 <layer number="44" name="Drills" color="7" fill="1" visible="no" active="no"/>
 <layer number="45" name="Holes" color="7" fill="1" visible="no" active="no"/>
-<layer number="46" name="Milling" color="3" fill="1" visible="yes" active="no"/>
-<layer number="47" name="Measures" color="7" fill="1" visible="yes" active="no"/>
-<layer number="48" name="Document" color="7" fill="1" visible="yes" active="no"/>
-<layer number="49" name="Reference" color="7" fill="1" visible="yes" active="no"/>
-<layer number="51" name="tDocu" color="7" fill="1" visible="yes" active="no"/>
-<layer number="52" name="bDocu" color="7" fill="1" visible="yes" active="no"/>
+<layer number="46" name="Milling" color="3" fill="1" visible="no" active="no"/>
+<layer number="47" name="Measures" color="7" fill="1" visible="no" active="no"/>
+<layer number="48" name="Document" color="7" fill="1" visible="no" active="no"/>
+<layer number="49" name="Reference" color="7" fill="1" visible="no" active="no"/>
+<layer number="51" name="tDocu" color="7" fill="1" visible="no" active="no"/>
+<layer number="52" name="bDocu" color="7" fill="1" visible="no" active="no"/>
 <layer number="90" name="Modules" color="5" fill="1" visible="yes" active="yes"/>
 <layer number="91" name="Nets" color="2" fill="1" visible="yes" active="yes"/>
@@
 <part name="C7" library="rcl" deviceset="C-EU" device="C0805" value="100n"/>
 <part name="U$2" library="foe-scale" deviceset="BAS521" device=""/>
+<part name="U$4" library="foe-scale" deviceset="RGBLED" device=""/>
+<part name="R16" library="resistor" deviceset="R-US_" device="R0805" value="15"/>
+<part name="R17" library="resistor" deviceset="R-US_" device="R0805" value="70"/>
+<part name="R18" library="resistor" deviceset="R-US_" device="R0805" value="15"/>
+<part name="SUPPLY19" library="supply2" deviceset="VDD" device="" value="3.3V"/>
+<part name="U$5" library="foe-scale" deviceset="BUZZER" device=""/>
+<part name="SUPPLY20" library="supply2" deviceset="GND" device=""/>
 </parts>
 <sheets>
@@
 <instance part="C7" gate="G$1" x="91.44" y="35.56"/>
 <instance part="U$2" gate="G$1" x="91.44" y="47.244"/>
+<instance part="U$4" gate="G$1" x="101.6" y="-53.34" rot="R90"/>
+<instance part="R16" gate="G$1" x="78.74" y="-63.5" rot="R180"/>
+<instance part="R17" gate="G$1" x="78.74" y="-53.34" rot="R180"/>
+<instance part="R18" gate="G$1" x="83.82" y="-58.42" rot="R180"/>
+<instance part="SUPPLY19" gate="G$1" x="111.76" y="-55.88"/>
+<instance part="U$5" gate="G$1" x="78.74" y="-43.18" rot="MR0"/>
+<instance part="SUPPLY20" gate="GND1" x="81.28" y="-45.72"/>
 </instances>
 <busses>
@@
 <wire x1="30.48" y1="101.6" x2="35.56" y2="101.6" width="0.1524" layer="91"/>
 <junction x="30.48" y="101.6"/>
+</segment>
+<segment>
+<pinref part="U$5" gate="G$1" pin="-"/>
+<pinref part="SUPPLY20" gate="GND1" pin="GND"/>
 </segment>
 </net>
@@
 <pinref part="SUPPLY13" gate="G$1" pin="VDD"/>
 </segment>
+<segment>
+<pinref part="U$4" gate="G$1" pin="A"/>
+<pinref part="SUPPLY19" gate="G$1" pin="VDD"/>
+</segment>
 </net>
 <net name="N$2" class="0">
@@
 </segment>
 </net>
+<net name="N$13" class="0">
+<segment>
+<pinref part="U1" gate="G$1" pin="PA22"/>
+<pinref part="R17" gate="G$1" pin="2"/>
+<wire x1="68.58" y1="-53.34" x2="73.66" y2="-53.34" width="0.1524" layer="91"/>
+</segment>
+</net>
+<net name="N$14" class="0">
+<segment>
+<pinref part="R18" gate="G$1" pin="2"/>
+<pinref part="U1" gate="G$1" pin="PA19"/>
+<wire x1="78.74" y1="-58.42" x2="68.58" y2="-58.42" width="0.1524" layer="91"/>
+</segment>
+</net>
+<net name="N$15" class="0">
+<segment>
+<pinref part="U1" gate="G$1" pin="PA18"/>
+<pinref part="R16" gate="G$1" pin="2"/>
+<wire x1="68.58" y1="-63.5" x2="73.66" y2="-63.5" width="0.1524" layer="91"/>
+</segment>
+</net>
+<net name="N$16" class="0">
+<segment>
+<pinref part="R16" gate="G$1" pin="1"/>
+<pinref part="U$4" gate="G$1" pin="4-GREEN"/>
+<wire x1="83.82" y1="-63.5" x2="96.52" y2="-63.5" width="0.1524" layer="91"/>
+</segment>
+</net>
+<net name="N$17" class="0">
+<segment>
+<pinref part="U$4" gate="G$1" pin="3-BLUE"/>
+<pinref part="R18" gate="G$1" pin="1"/>
+<wire x1="96.52" y1="-58.42" x2="88.9" y2="-58.42" width="0.1524" layer="91"/>
+</segment>
+</net>
+<net name="N$18" class="0">
+<segment>
+<pinref part="R17" gate="G$1" pin="1"/>
+<pinref part="U$4" gate="G$1" pin="1-RED"/>
+<wire x1="83.82" y1="-53.34" x2="96.52" y2="-53.34" width="0.1524" layer="91"/>
+</segment>
+</net>
+<net name="N$19" class="0">
+<segment>
+<pinref part="U1" gate="G$1" pin="PA23"/>
+<pinref part="U$5" gate="G$1" pin="+"/>
+<wire x1="68.58" y1="-48.26" x2="73.66" y2="-48.26" width="0.1524" layer="91"/>
+<wire x1="73.66" y1="-48.26" x2="73.66" y2="-43.18" width="0.1524" layer="91"/>
+</segment>
+</net>
+<net name="ENVSENSE" class="0">
+<segment>
+<pinref part="U1" gate="G$1" pin="PA06"/>
+<wire x1="7.62" y1="-63.5" x2="-7.62" y2="-63.5" width="0.1524" layer="91"/>
+<label x="-7.62" y="-63.5" size="1.778" layer="95"/>
+</segment>
+</net>
+<net name="CARSENSE" class="0">
+<segment>
+<pinref part="U1" gate="G$1" pin="PA05"/>
+<wire x1="7.62" y1="-58.42" x2="-7.62" y2="-58.42" width="0.1524" layer="91"/>
+<label x="-7.62" y="-58.42" size="1.778" layer="95"/>
+</segment>
+</net>
+<net name="IMON" class="0">
+<segment>
+<pinref part="U1" gate="G$1" pin="PA04"/>
+<wire x1="7.62" y1="-53.34" x2="-7.62" y2="-53.34" width="0.1524" layer="91"/>
+<label x="-7.62" y="-53.34" size="1.778" layer="95"/>
+</segment>
+</net>
+<net name="ALIGNED" class="0">
+<segment>
+<pinref part="U1" gate="G$1" pin="PA03"/>
+<wire x1="7.62" y1="-48.26" x2="-7.62" y2="-48.26" width="0.1524" layer="91"/>
+<label x="-7.62" y="-48.26" size="1.778" layer="95"/>
+</segment>
+</net>
